File: Advanced-PCB/Fluff-Advanced-PCB-master/Fluff-Advanced-PCB-master/Advanced-PCB/Advanced-PCB.sch (KiCad schematic (older format))
At the start: 154 parts, among them J1 USB_mini_micro_B, SW1 Esc, SW10 Win 1.25, SW11 2, SW12 W, SW13 S, SW14 X, SW15 Alt 1.25, SW16 3, SW17 E, SW18 D, SW19 C, SW2 Tab 1.50, SW20 4, SW21 R, SW22 F, SW23 V, SW24 5, SW25 T, SW26 G, SW27 B, SW28 Space 6.25, SW29 6, SW3 Caps 1.75, SW30 Y, SW31 H, SW32 N, SW33 7, SW34 U, SW35 J, SW36 M, SW37 8, SW38 I, SW39 K, SW4 Shift 2.25, SW40 ,, SW41 9, SW42 P, SW43 L, SW44 ., SW45 Alt 1.25, SW46 0, SW47 O, SW48 ;, SW49 /, SW5 Ctrl 1.25, SW50 Fn 1.25, SW51 -, SW52 [, SW53 ', SW54 Shift 1.75, SW55 Left Arrow, SW56 =, SW57 ], SW58 Enter 2.25, SW59 Up Arrow, SW6 1, SW60 Down Arrow, SW61 Back 2.00, SW62 \\ 1.50, SW63 Pg Up, SW64 Pg Down, SW65 Right Arrow, SW66 `, SW67 Del, SW68 Alt 1.00, SW69 Fn 1.00, SW7 Q, SW70 Ctrl 1.00, SW8 A, SW9 Z, U1 ATMEGA32U4, X1 XTAL_GND

Commit message: PCB-Rerouted
Correctly Rerouted and except of errors except for with layer keys.
Parts:
- SW1: footprint acheron_MX:MX100 -> acheron_MXA:MXA100
- SW2: footprint acheron_MX:MX150 -> acheron_MXA:MXA150
- SW3: footprint acheron_MX:MX175 -> acheron_MXA:MXA175
- SW4: footprint acheron_MX:MX225R -> acheron_MXA:MXA225R
- SW5: footprint acheron_MX:MX125 -> acheron_MXA:MXA125
Connections:
- net Col1: now also U1.11 (PB3/MISO); no longer U1.41 (PF0)
- net Col10: now also U1.32 (PC7); no longer U1.30 (PB6)
- net Col11: now also U1.22 (PD5/XCK1); no longer U1.25 (ICP1/PD4)
- net Col12: now also U1.21 (PD3/TXD1); no longer U1.26 (T1/PD6)
- net Col13: now also U1.20 (PD2/RXD1); no longer U1.27 (T0/PD7)
- net Col14: now also U1.19 (PD1/INT1); no longer U1.28 (PB4)
- net Col15: now also U1.18 (PD0/INT0); no longer U1.29 (PB5)
- net Col2: now also U1.36 (PF7); no longer U1.40 (PF1)
- net Col3: now also U1.25 (ICP1/PD4); no longer U1.39 (PF4)
- net Col4: now also U1.26 (T1/PD6); no longer U1.38 (PF5)
- net Col5: now also U1.27 (T0/PD7); no longer U1.37 (PF6)
- net Col6: now also U1.28 (PB4); no longer U1.11 (PB3/MISO)
- net Col7: now also U1.29 (PB5); no longer U1.36 (PF7)
- net Col8: now also U1.30 (PB6); no longer U1.32 (PC7)
- net Row0: now also U1.40 (PF1); no longer U1.42 (AREF)
- net Row1: now also U1.41 (PF0); no longer U1.22 (PD5/XCK1)
- net Row2: now also U1.39 (PF4); no longer U1.21 (PD3/TXD1)
- net Row3: now also U1.38 (PF5); no longer U1.20 (PD2/RXD1)
- net Row4: now also U1.37 (PF6); no longer U1.19 (PD1/INT1)
- net at D46.2 (A): no longer SW46.2 (Row)
- no-connect marks 7 -> 6
Other:
- moved on the sheet: D46
Changed lines of the file:
@@
 	10900 1000 10900 1250
 Connection ~ 9700 1775
+Connection ~ 10050 1000
+Wire Wire Line
+	10050 1000 10050 1275
 $Comp
 L Device:D_Small D51
@@
 L Device:D_Small D46
 U 1 1 5E834C3E
-P 10050 1325
-F 0 "D46" V 10125 1375 50  0000 L CNN
-F 1 "1N4148W" V 9925 1200 50  0000 L CNN
-F 2 "Diode_SMD:D_SOD-123" V 10050 1325 50  0001 C CNN
-F 3 "~" V 10050 1325 50  0001 C CNN
-	1    10050 1325
+P 10050 1375
+F 0 "D46" V 10125 1425 50  0000 L CNN
+F 1 "1N4148W" V 9925 1250 50  0000 L CNN
+F 2 "Diode_SMD:D_SOD-123" V 10050 1375 50  0001 C CNN
+F 3 "~" V 10050 1375 50  0001 C CNN
+	1    10050 1375
 	0    1    1    0
 $EndComp
@@
 F 0 "SW1" H 1525 1875 50  0000 L CNN
 F 1 "Esc" H 1600 1775 79  0000 C CNN
-F 2 "acheron_MX:MX100" H 1600 1775 50  0001 C CNN
+F 2 "acheron_MXA:MXA100" H 1600 1775 50  0001 C CNN
 F 3 "" H 1600 1775 50  0001 C CNN
 	1    1600 1775
@@
 F 0 "SW2" H 1525 3100 50  0000 L CNN
 F 1 "Tab 1.50" H 1600 3000 59  0000 C CNN
-F 2 "acheron_MX:MX150" H 1600 3000 50  0001 C CNN
+F 2 "acheron_MXA:MXA150" H 1600 3000 50  0001 C CNN
 F 3 "" H 1600 3000 50  0001 C CNN
 	1    1600 3000
@@
 F 0 "SW3" H 1525 4275 50  0000 L CNN
 F 1 "Caps 1.75" H 1600 4175 59  0000 C CNN
-F 2 "acheron_MX:MX175" H 1600 4175 50  0001 C CNN
+F 2 "acheron_MXA:MXA175" H 1600 4175 50  0001 C CNN
 F 3 "" H 1600 4175 50  0001 C CNN
 	1    1600 4175
@@
 F 0 "SW4" H 1525 5500 50  0000 L CNN
 F 1 "Shift 2.25" H 1600 5400 59  0000 C CNN
-F 2 "acheron_MX:MX225R" H 1600 5400 50  0001 C CNN
+F 2 "acheron_MXA:MXA225R" H 1600 5400 50  0001 C CNN
 F 3 "" H 1600 5400 50  0001 C CNN
 	1    1600 5400
@@
 F 0 "SW5" H 1525 6725 50  0000 L CNN
 F 1 "Ctrl 1.25" H 1600 6625 59  0000 C CNN
-F 2 "acheron_MX:MX125" H 1600 6625 50  0001 C CNN
+F 2 "acheron_MXA:MXA125" H 1600 6625 50  0001 C CNN
 F 3 "" H 1600 6625 50  0001 C CNN
 	1    1600 6625
@@
 	10125 6275 10050 6275
 NoConn ~ 5275 13475
-Text GLabel 2850 15375 2    50   Input ~ 0
+Text GLabel 5550 13575 0    50   Input ~ 0
 Row1
 Wire Wire Line
-	5275 13575 5550 13575
-Text GLabel 5550 13775 0    50   Input ~ 0
+	3125 14275 2850 14275
+Text GLabel 5550 15175 0    50   Input ~ 0
 Col3
-Text GLabel 5550 13875 0    50   Input ~ 0
+Text GLabel 5550 15075 0    50   Input ~ 0
 Col4
-Text GLabel 5550 13975 0    50   Input ~ 0
+Text GLabel 5550 14975 0    50   Input ~ 0
 Col5
-Text GLabel 2850 14275 2    50   Input ~ 0
+Text GLabel 5550 14875 0    50   Input ~ 0
 Col6
 Text GLabel 5550 14575 0    50   Input ~ 0
 Col9
-Text GLabel 5550 14475 0    50   Input ~ 0
+Text GLabel 5550 14675 0    50   Input ~ 0
 Col8
-Text GLabel 5550 14075 0    50   Input ~ 0
+Text GLabel 5550 14775 0    50   Input ~ 0
 Col7
 $Comp
@@
 $EndComp
 Wire Wire Line
-	5275 13775 5550 13775
-Wire Wire Line
-	5275 13875 5550 13875
-Wire Wire Line
-	5275 13975 5550 13975
-Wire Wire Line
-	3125 14275 2850 14275
+	5275 15175 5550 15175
+Wire Wire Line
+	5275 15075 5550 15075
+Wire Wire Line
+	5275 14975 5550 14975
+Wire Wire Line
+	5275 14875 5550 14875
 Wire Wire Line
 	5275 14575 5550 14575
 Wire Wire Line
-	5275 14475 5550 14475
-Wire Wire Line
-	5275 14075 5550 14075
-Text GLabel 5600 14675 0    50   Input ~ 0
+	5275 14675 5550 14675
+Wire Wire Line
+	5275 14775 5550 14775
+Text GLabel 5600 14475 0    50   Input ~ 0
 Col10
-Text GLabel 5525 14775 0    50   Input ~ 0
+Text GLabel 2875 14975 2    50   Input ~ 0
 Col15
-Text GLabel 5525 14875 0    50   Input ~ 0
+Text GLabel 2875 15075 2    50   Input ~ 0
 Col14
-Text GLabel 5525 14975 0    50   Input ~ 0
+Text GLabel 2875 15175 2    50   Input ~ 0
 Col13
-Text GLabel 5525 15075 0    50   Input ~ 0
+Text GLabel 2875 15275 2    50   Input ~ 0
 Col12
-Wire Wire Line
-	5525 15075 5275 15075
-Wire Wire Line
-	5525 14975 5275 14975
-Wire Wire Line
-	5525 14875 5275 14875
-Wire Wire Line
-	5525 14775 5275 14775
+Text GLabel 2875 15375 2    50   Input ~ 0
+Col11
+Wire Wire Line
+	2875 15375 3125 15375
+Wire Wire Line
+	2875 15275 3125 15275
+Wire Wire Line
+	2875 15175 3125 15175
+Wire Wire Line
+	2875 15075 3125 15075
+Wire Wire Line
+	2875 14975 3125 14975
 Connection ~ 13050 1775
 Wire Wire Line
@@
 Wire Wire Line
 	9700 825  9700 1775
+Wire Wire Line
+	9200 1000 10050 1000
 Connection ~ 10550 1800
 Wire Wire Line
 	10550 825  10550 1800
+Wire Wire Line
+	10050 1000 10900 1000
 Wire Wire Line
 	11350 825  11350 1775
@@
 	1500 14125 1775 14125
 Wire Wire Line
-	5275 14675 5600 14675
+	5275 14475 5600 14475
 $Comp
 L Device:R R4
@@
 	0    1    1    0
 $EndComp
-Text GLabel 5550 13675 0    50   Input ~ 0
+Text GLabel 5550 14075 0    50   Input ~ 0
 Col2
 Wire Wire Line
-	5275 13675 5550 13675
+	5275 14075 5550 14075
 $Comp
 L power:GND #PWR0108
@@
 	0    -1   -1   0
 $EndComp
-Text GLabel 5550 13575 0    50   Input ~ 0
+Text GLabel 2850 14275 2    50   Input ~ 0
 Col1
 Wire Wire Line
-	3125 15075 2850 15075
-Wire Wire Line
-	3125 15175 2850 15175
-Wire Wire Line
-	3125 15275 2850 15275
-Text GLabel 2850 15075 2    50   Input ~ 0
+	5275 13975 5550 13975
+Wire Wire Line
+	5275 13875 5550 13875
+Wire Wire Line
+	5275 13775 5550 13775
+Wire Wire Line
+	5275 13675 5550 13675
+Text GLabel 5550 13975 0    50   Input ~ 0
 Row4
-Text GLabel 2850 15175 2    50   Input ~ 0
+Text GLabel 5550 13875 0    50   Input ~ 0
 Row3
-Text GLabel 2850 15275 2    50   Input ~ 0
+Text GLabel 5550 13775 0    50   Input ~ 0
 Row2
-Wire Wire Line
-	3125 15375 2850 15375
-Wire Wire Line
-	9200 1000 10050 1000
-Wire Wire Line
-	10050 1225 10050 1000
-Connection ~ 10050 1000
-Wire Wire Line
-	10050 1000 10900 1000
-Wire Wire Line
-	5275 13475 5550 13475
-Text GLabel 5550 13475 0    50   Input ~ 0
+Text GLabel 5550 13675 0    50   Input ~ 0
 Row0
 Wire Wire Line
-	5525 15175 5275 15175
-Text GLabel 5525 15175 0    50   Input ~ 0
-Col11
-NoConn ~ 3125 14975
+	5275 13575 5550 13575
 $EndSCHEMATC
