File: Advanced-PCB/Advanced-PCB.kicad_pcb (KiCad board)
At the start: 2 copper layers, 318.9 x 109.4 mm, 154 parts, among them J1 USB_mini_micro_B, SW1 Esc, SW10 Win 1.25, SW11 2, SW12 W, SW13 S, SW14 X, SW15 Alt 1.25, SW16 3, SW17 E, SW18 D, SW19 C, SW2 Tab 1.50, SW20 4, SW21 R, SW22 F, SW23 V, SW24 5, SW25 T, SW26 G, SW27 B, SW28 Space 6.25, SW29 6, SW3 Caps 1.75, SW30 Y, SW31 H, SW32 N, SW33 7, SW34 U, SW35 J, SW36 M, SW37 8, SW38 I, SW39 K, SW4 Shift 2.25, SW40 ,, SW41 9, SW42 P, SW43 L, SW44 ., SW45 Alt 1.25, SW46 0, SW47 O, SW48 ;, SW49 /, SW5 Ctrl 1.25, SW50 Fn 1.25, SW51 -, SW52 [, SW53 ', SW54 Shift 1.75, SW55 Left Arrow, SW56 =, SW57 ], SW58 Enter 2.25, SW59 Up Arrow, SW6 1, SW60 Down Arrow, SW61 Back 2.00, SW62 \ 1.50, SW63 Pg Up, SW64 Pg Down, SW65 Right Arrow, SW66 `, SW67 Del, SW68 Alt 1.00, SW69 Fn 1.00, SW7 Q, SW70 Ctrl 1.00, SW8 A, SW9 Z, U1 ATMEGA32U4, X1 XTAL_GND

Commit message: BACKUP
Parts:
- removed C8: 1u, Capacitor_SMD:C_0805_2012Metric_Pad1.15x1.40mm_HandSolder
- removed J1: USB_mini_micro_B, acheron_Connectors:USB_MiniB_Hirose_UX60-MB-5S8
- removed R2, R3: 22, Resistor_SMD:R_0805_2012Metric_Pad1.15x1.40mm_HandSolder
- added C23: 1u, Capacitor_SMD:C_0603_1608Metric, F.Cu at (277.1, 7.08)
- added F2: 500mA, Resistor_SMD:R_0805_2012Metric, F.Cu at (277.3, 4.35)
- added LED100: LED, LED_SMD:LED_WS2812B_PLCC4_5.0x5.0mm_P3.2mm, F.Cu at (313.0, -7.06)
- added LED101: LED, LED_SMD:LED_WS2812B_PLCC4_5.0x5.0mm_P3.2mm, F.Cu at (348.9, -40.2)
- added LED102: LED, LED_SMD:LED_WS2812B_PLCC4_5.0x5.0mm_P3.2mm, F.Cu at (321.4, -13.7)
- added LED103: LED, LED_SMD:LED_WS2812B_PLCC4_5.0x5.0mm_P3.2mm, F.Cu at (329.8, -20.3)
- added LED104: LED, LED_SMD:LED_WS2812B_PLCC4_5.0x5.0mm_P3.2mm, F.Cu at (338.2, -26.9)
- added LED105: LED, LED_SMD:LED_WS2812B_PLCC4_5.0x5.0mm_P3.2mm, F.Cu at (313.0, -0.44)
- added LED106: LED, LED_SMD:LED_WS2812B_PLCC4_5.0x5.0mm_P3.2mm, F.Cu at (348.9, -33.5)
- added LED107: LED, LED_SMD:LED_WS2812B_PLCC4_5.0x5.0mm_P3.2mm, F.Cu at (321.4, -7.06)
- added LED108: LED, LED_SMD:LED_WS2812B_PLCC4_5.0x5.0mm_P3.2mm, F.Cu at (304.6, -0.44)
- added LED109: LED, LED_SMD:LED_WS2812B_PLCC4_5.0x5.0mm_P3.2mm, F.Cu at (323.6, -40.2)
- added LED110: LED, LED_SMD:LED_WS2812B_PLCC4_5.0x5.0mm_P3.2mm, F.Cu at (340.5, -33.5)
- added LED111: LED, LED_SMD:LED_WS2812B_PLCC4_5.0x5.0mm_P3.2mm, F.Cu at (346.7, -26.9)
- added LED112: LED, LED_SMD:LED_WS2812B_PLCC4_5.0x5.0mm_P3.2mm, F.Cu at (321.4, -0.44)
- added LED113: LED, LED_SMD:LED_WS2812B_PLCC4_5.0x5.0mm_P3.2mm, F.Cu at (329.8, -7.06)
- added LED114: LED, LED_SMD:LED_WS2812B_PLCC4_5.0x5.0mm_P3.2mm, F.Cu at (338.2, -13.7)
- added LED115: LED, LED_SMD:LED_WS2812B_PLCC4_5.0x5.0mm_P3.2mm, F.Cu at (346.7, -20.3)
- added LED116: LED, LED_SMD:LED_WS2812B_PLCC4_5.0x5.0mm_P3.2mm, F.Cu at (355.1, -26.9)
- added LED117: LED, LED_SMD:LED_WS2812B_PLCC4_5.0x5.0mm_P3.2mm, F.Cu at (338.2, -0.44)
- added LED118: LED, LED_SMD:LED_WS2812B_PLCC4_5.0x5.0mm_P3.2mm, F.Cu at (329.8, -13.7)
- added LED119: LED, LED_SMD:LED_WS2812B_PLCC4_5.0x5.0mm_P3.2mm, F.Cu at (338.2, -7.06)
- added LED120: LED, LED_SMD:LED_WS2812B_PLCC4_5.0x5.0mm_P3.2mm, F.Cu at (346.7, -13.7)
- added LED121: LED, LED_SMD:LED_WS2812B_PLCC4_5.0x5.0mm_P3.2mm, F.Cu at (355.1, -20.3)
- added LED52: LED, LED_SMD:LED_WS2812B_PLCC4_5.0x5.0mm_P3.2mm, F.Cu at (270.9, -9.63)
- added LED53: LED, LED_SMD:LED_WS2812B_PLCC4_5.0x5.0mm_P3.2mm, F.Cu at (281.5, -40.2)
- added LED54: LED, LED_SMD:LED_WS2812B_PLCC4_5.0x5.0mm_P3.2mm, F.Cu at (270.9, -22.9)
- added LED55: LED, LED_SMD:LED_WS2812B_PLCC4_5.0x5.0mm_P3.2mm, F.Cu at (281.5, -33.5)
- added LED56: LED, LED_SMD:LED_WS2812B_PLCC4_5.0x5.0mm_P3.2mm, F.Cu at (289.9, -40.2)
- added LED57: LED, LED_SMD:LED_WS2812B_PLCC4_5.0x5.0mm_P3.2mm, F.Cu at (270.9, -16.2)
- added LED58: LED, LED_SMD:LED_WS2812B_PLCC4_5.0x5.0mm_P3.2mm, F.Cu at (279.3, -26.9)
- added LED59: LED, LED_SMD:LED_WS2812B_PLCC4_5.0x5.0mm_P3.2mm, F.Cu at (296.1, -26.9)
- added LED60: LED, LED_SMD:LED_WS2812B_PLCC4_5.0x5.0mm_P3.2mm, F.Cu at (298.4, -40.2)
- added LED61: LED, LED_SMD:LED_WS2812B_PLCC4_5.0x5.0mm_P3.2mm, F.Cu at (270.9, -29.5)
- added LED62: LED, LED_SMD:LED_WS2812B_PLCC4_5.0x5.0mm_P3.2mm, F.Cu at (287.7, -26.9)
- added LED63: LED, LED_SMD:LED_WS2812B_PLCC4_5.0x5.0mm_P3.2mm, F.Cu at (279.3, -20.3)
- added LED64: LED, LED_SMD:LED_WS2812B_PLCC4_5.0x5.0mm_P3.2mm, F.Cu at (298.4, -33.5)
- added LED65: LED, LED_SMD:LED_WS2812B_PLCC4_5.0x5.0mm_P3.2mm, F.Cu at (306.8, -40.2)
- added LED66: LED, LED_SMD:LED_WS2812B_PLCC4_5.0x5.0mm_P3.2mm, F.Cu at (279.3, -13.7)
- added LED67: LED, LED_SMD:LED_WS2812B_PLCC4_5.0x5.0mm_P3.2mm, F.Cu at (270.9, -3.01)
- added LED68: LED, LED_SMD:LED_WS2812B_PLCC4_5.0x5.0mm_P3.2mm, F.Cu at (287.7, -20.3)
- added LED69: LED, LED_SMD:LED_WS2812B_PLCC4_5.0x5.0mm_P3.2mm, F.Cu at (289.9, -33.5)
- added LED70: LED, LED_SMD:LED_WS2812B_PLCC4_5.0x5.0mm_P3.2mm, F.Cu at (279.3, -7.06)
- added LED71: LED, LED_SMD:LED_WS2812B_PLCC4_5.0x5.0mm_P3.2mm, F.Cu at (315.2, -40.2)
- added LED72: LED, LED_SMD:LED_WS2812B_PLCC4_5.0x5.0mm_P3.2mm, F.Cu at (287.7, -13.7)
- added LED73: LED, LED_SMD:LED_WS2812B_PLCC4_5.0x5.0mm_P3.2mm, F.Cu at (27.1, 138.6)
- added LED74: LED, LED_SMD:LED_WS2812B_PLCC4_5.0x5.0mm_P3.2mm, F.Cu at (296.1, -20.3)
- added LED75: LED, LED_SMD:LED_WS2812B_PLCC4_5.0x5.0mm_P3.2mm, F.Cu at (304.6, -26.9)
- added LED76: LED, LED_SMD:LED_WS2812B_PLCC4_5.0x5.0mm_P3.2mm, F.Cu at (279.3, -0.44)
- added LED77: LED, LED_SMD:LED_WS2812B_PLCC4_5.0x5.0mm_P3.2mm, F.Cu at (315.2, -33.5)
- added LED78: LED, LED_SMD:LED_WS2812B_PLCC4_5.0x5.0mm_P3.2mm, F.Cu at (304.6, -13.7)
- added LED79: LED, LED_SMD:LED_WS2812B_PLCC4_5.0x5.0mm_P3.2mm, F.Cu at (287.7, -7.06)
- added LED80: LED, LED_SMD:LED_WS2812B_PLCC4_5.0x5.0mm_P3.2mm, F.Cu at (306.8, -33.5)
- added LED81: LED, LED_SMD:LED_WS2812B_PLCC4_5.0x5.0mm_P3.2mm, F.Cu at (296.1, -13.7)
- added LED82: LED, LED_SMD:LED_WS2812B_PLCC4_5.0x5.0mm_P3.2mm, F.Cu at (304.6, -20.3)
- added LED83: LED, LED_SMD:LED_WS2812B_PLCC4_5.0x5.0mm_P3.2mm, F.Cu at (313.0, -26.9)
- added LED84: LED, LED_SMD:LED_WS2812B_PLCC4_5.0x5.0mm_P3.2mm, F.Cu at (287.7, -0.44)
- added LED85: LED, LED_SMD:LED_WS2812B_PLCC4_5.0x5.0mm_P3.2mm, F.Cu at (323.6, -33.5)
- added LED86: LED, LED_SMD:LED_WS2812B_PLCC4_5.0x5.0mm_P3.2mm, F.Cu at (296.1, -7.06)
- added LED87: LED, LED_SMD:LED_WS2812B_PLCC4_5.0x5.0mm_P3.2mm, F.Cu at (332.0, -40.2)
- added LED88: LED, LED_SMD:LED_WS2812B_PLCC4_5.0x5.0mm_P3.2mm, F.Cu at (329.8, -0.44)
- added LED89: LED, LED_SMD:LED_WS2812B_PLCC4_5.0x5.0mm_P3.2mm, F.Cu at (346.7, -7.06)
- added LED90: LED, LED_SMD:LED_WS2812B_PLCC4_5.0x5.0mm_P3.2mm, F.Cu at (321.4, -26.9)
- added LED91: LED, LED_SMD:LED_WS2812B_PLCC4_5.0x5.0mm_P3.2mm, F.Cu at (296.1, -0.44)
- added LED92: LED, LED_SMD:LED_WS2812B_PLCC4_5.0x5.0mm_P3.2mm, F.Cu at (332.0, -33.5)
- added LED93: LED, LED_SMD:LED_WS2812B_PLCC4_5.0x5.0mm_P3.2mm, F.Cu at (304.6, -7.06)
- added LED94: LED, LED_SMD:LED_WS2812B_PLCC4_5.0x5.0mm_P3.2mm, F.Cu at (340.5, -40.2)
- added LED95: LED, LED_SMD:LED_WS2812B_PLCC4_5.0x5.0mm_P3.2mm, F.Cu at (313.0, -13.7)
- added LED96: LED, LED_SMD:LED_WS2812B_PLCC4_5.0x5.0mm_P3.2mm, F.Cu at (321.4, -20.3)
- added LED97: LED, LED_SMD:LED_WS2812B_PLCC4_5.0x5.0mm_P3.2mm, F.Cu at (329.8, -26.9)
- added LED98: LED, LED_SMD:LED_WS2812B_PLCC4_5.0x5.0mm_P3.2mm, F.Cu at (338.2, -20.3)
- added LED99: LED, LED_SMD:LED_WS2812B_PLCC4_5.0x5.0mm_P3.2mm, F.Cu at (313.0, -20.3)
- added R10: 5.1k, Resistor_SMD:R_0603_1608Metric, F.Cu at (285.5, 6.64)
- added R7: 22, Resistor_SMD:R_0603_1608Metric, F.Cu at (281.5, 4.13)
- added R8: 22, Resistor_SMD:R_0603_1608Metric, F.Cu at (281.5, 6.64)
- added R9: 5.1k, Resistor_SMD:R_0603_1608Metric, F.Cu at (285.5, 4.13)
- added USB2: HRO-TYPE-C-31-M-12, Type-C_Master:HRO-TYPE-C-31-M-12-HandSoldering, F.Cu at (272.0, -33.5)
- D1, D10, D11, D12, D13, D14, D15, D16, D17, D18, D19, D2, D20, D21, D22, D23, D24, D25, D26, D27, D28, D29, D3, D30, D31, D32, D33, D34, D35, D36, D37, D38, D39, D4, D40, D41, D42, D43, D44, D45, D46, D47, D48, D49, D5, D50, D51, D52, D53, D54, D55, D56, D57, D58, D59, D6, D60, D61, D62, D63, D64, D65, D66, D67, D7, D70, D8, D9: footprint Diode_SMD:D_SOD-123 -> keyboard-parts:D_SOD123_axial
- SW70: footprint acheron_MXA:MXA100 -> acheron_MX:MX100
- moved D50 15.4 mm to (227.2, 134.8), turned to 90 degrees
- moved D45 10.7 mm to (208.2, 134.8), turned to 90 degrees
- moved D36 9.67 mm to (174.8, 113.5), turned to 90 degrees
- moved D4 9.52 mm to (28.8, 115.0), turned to 90 degrees
- moved D58 9.02 mm to (272.0, 96.5), turned to 90 degrees
- moved D61 8.89 mm to (274.5, 58.5), turned to 90 degrees
- moved D3 8.89 mm to (24.5, 96.8), turned to 90 degrees
- moved D5 8.87 mm to (19.8, 134.8), turned to 90 degrees
- moved D44 8.85 mm to (212.8, 115.2), turned to 90 degrees
- moved D54 8.85 mm to (258.0, 115.2), turned to 90 degrees
- moved D64 8.85 mm to (303.2, 115.2), turned to 90 degrees
- moved D59 8.80 mm to (284.2, 115.2), turned to 90 degrees
- moved D35 8.79 mm to (165.0, 96.8), turned to 90 degrees
- moved D17 8.79 mm to (84.0, 77.8), turned to 90 degrees
- moved D27 8.76 mm to (136.5, 115.8), turned to 90 degrees
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Connections:
- net Net-(U1-Pad8) renamed LED_PWM
- U1 pad 18: Net-(U1-Pad18) -> Row0
- U1 pad 2: VCC -> +5V
- U1 pad 42: Row0 -> Net-(U1-Pad42)
- U1 pad 7: VCC -> +5V
Routing:
- net Col2: track 778.4 -> 406.8 mm, vias 0 -> 2
- net Net-(D40-Pad2): track 9.49 -> 41.4 mm, vias 0 -> 2
- net GND: track 376.7 -> 408.2 mm, vias 13 -> 16
- net Net-(D70-Pad2): track 9.49 -> 24.8 mm, vias 0 -> 2
- net Net-(D6-Pad2): track 9.53 -> 24.1 mm, vias 0 -> 2
- net Col4: track 412.5 -> 424.1 mm, vias 0 -> 2
- net Col5: track 433.7 -> 445.2 mm, vias 0 -> 2
- net Col7: track 477.9 -> 489.0 mm, vias 0 -> 3
- net Row2: track 384.2 -> 395.1 mm
- net Net-(D45-Pad2): track 17.3 -> 8.90 mm
- net Col3: track 423.5 -> 431.9 mm, vias 0 -> 4
- net Net-(D50-Pad2): track 18.4 -> 11.9 mm
- net Row1: track 344.9 -> 339.8 mm, vias 18 -> 16
- net Net-(J1-Pad3): track 8.46 -> 13.5 mm
- net Row3: track 420.6 -> 415.7 mm
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Other:
- outline, holes or cut-outs redrawn
- net class Default: via_dia 0.8 -> 0.4445
