File: Advanced-PCB/Without Led and Usb-c.kicad_pcb (KiCad board)
At the start: 2 copper layers, 318.9 x 109.4 mm, 160 parts, among them J1 USB_mini_micro_B, SW1 Esc, SW10 Win 1.25, SW11 2, SW12 W, SW13 S, SW14 X, SW15 Alt 1.25, SW16 3, SW17 E, SW18 D, SW19 C, SW2 Tab 1.50, SW20 4, SW21 R, SW22 F, SW23 V, SW24 5, SW25 T, SW26 G, SW27 B, SW28 Space 6.25, SW29 6, SW3 Caps 1.75, SW30 Y, SW31 H, SW32 N, SW33 7, SW34 U, SW35 J, SW36 M, SW37 8, SW38 I, SW39 K, SW4 Shift 2.25, SW40 ,, SW41 9, SW42 P, SW43 L, SW44 ., SW45 Alt 1.25, SW46 0, SW47 O, SW48 ;, SW49 /, SW5 Ctrl 1.25, SW50 Fn 1.25, SW51 -, SW52 [, SW53 ', SW54 Shift 1.75, SW55 Left Arrow, SW56 =, SW57 ], SW58 Enter 2.25, SW59 Up Arrow, SW6 1, SW60 Down Arrow, SW61 Back 2.00, SW62 \ 1.50, SW63 Pg Up, SW64 Pg Down, SW65 Right Arrow, SW66 `, SW67 Del, SW68 Alt 1.00, SW69 Fn 1.00, SW7 Q, SW70 Ctrl 1.00, SW8 A, SW9 Z, U1 ATMEGA32U4, X1 XTAL_GND

Commit message: BACKUP
Parts:
- added G***: LOGO, Teddy:Fluff, F.Cu at (297.6, 139.9)
- added G***: LOGO, Teddy:Teddy2, F.Cu at (62.7, 101.8)
